File: hardware/reDIP-SID.sch (KiCad schematic (older format))
At the start: 72 parts, among them J1 Conn_01x01, J2 Conn_01x05, J3 Conn_01x14, J4 Conn_01x10, J5 TYPE-C-31-M-12, J6 Conn_02x05_Odd_Even, SW1 KXT311LHS, U1 NCP115AMX120TCG, U10 W25Q128JVPIM, U11 ICE40UP5K-SG48I, U2 NCP167AMX330TBG, U3 NCP115AMX120TCG, U4 FPF1321UCX, U5 SN74CBTD16211DGVR, U6 SGTL5000XNLA3, U7 NUF2042XV6, U8 MCP6H01T-E/OT, U9 LY68L6400SLIT, X1 ASCO-24.000MHZ-EK-T3

Commit message: Added silkscreen polarity marking for tantalum capacitors
Parts:
- C14, C15: footprint Capacitor_SMD:C_0603_1608Metric -> Capacitor_Tantalum_SMD:CP_EIA-1608-08_AVX-J
Changed lines of the file:
@@
 F 0 "C14" V 10600 3100 50  0000 C CNN
 F 1 "10uF" V 10600 2850 50  0000 C CNN
-F 2 "Capacitor_SMD:C_0603_1608Metric" H 10550 3000 50  0001 C CNN
+F 2 "Capacitor_Tantalum_SMD:CP_EIA-1608-08_AVX-J" H 10550 3000 50  0001 C CNN
 F 3 "https://www.vishay.com/docs/40176/tmcj.pdf" H 10550 3000 50  0001 C CNN
 F 4 "Vishay" H 10550 3000 50  0001 C CNN "Mfg"
@@
 F 0 "C15" V 10600 3300 50  0000 C CNN
 F 1 "10uF" V 10600 3050 50  0000 C CNN
-F 2 "Capacitor_SMD:C_0603_1608Metric" H 10550 3200 50  0001 C CNN
+F 2 "Capacitor_Tantalum_SMD:CP_EIA-1608-08_AVX-J" H 10550 3200 50  0001 C CNN
 F 3 "https://www.vishay.com/docs/40176/tmcj.pdf" H 10550 3200 50  0001 C CNN
 F 4 "Vishay" H 10550 3200 50  0001 C CNN "Mfg"
